Commit message: a radius is actually half of a diamater

File: ugv_description/urdf/choo_choo/model.urdf.xacro (robot description, xacro)
@@ -26,5 +26,5 @@
     <xacro:property name="lidar_mass" value="0.830" />
     <xacro:property name="lidar_height" value="0.0717" />
-    <xacro:property name="lidar_radius" value="0.1033" />
+    <xacro:property name="lidar_radius" value="0.0516" />
     <!-- imu properties -->
     <xacro:property name="imu_offset_x" value="0.0" />

Commit message: adjusts namespaces and topics

File: ugv_description/urdf/choo_choo/model.urdf.xacro (robot description, xacro)
@@ -1,4 +1,5 @@
 <?xml version="1.0"?>
 <robot xmlns:xacro="http://www.ros.org/wiki/xacro" name="choo_choo">
+    <xacro:property name="robot" value="choo_choo"/>
     <!-- physical parameters of robot, all in SI (meters, kg) -->
     <!-- base dimensions -->
@@ -9,5 +10,5 @@
     <!-- wheel properties -->
     <xacro:property name="wheel_radius" value="0.10795" />
-    <xacro:property name="wheel_width" value="0.061" />
+    <xacro:property name="wheel_width" value="0.059" />
     <!-- differential properties -->
     <xacro:property name="wheel_mass" value="1.179" />
@@ -89,4 +90,14 @@
                 <material>Gazebo/Black</material>
                 <gravity>true</gravity>
+                <surface>
+                    <friction>
+                        <ode>
+                            <mu>1</mu>
+                            <mu2>0</mu2>
+                            <fdir1>0 1.0 0</fdir1>
+                            <implicit_spring_damper>true</implicit_spring_damper>
+                        </ode>
+                    </friction>
+                </surface>
             </gazebo>
             <collision name="${name}_collision">
@@ -201,6 +212,7 @@
             <visualize>false</visualize>
             <plugin name="laser_plugin" filename="libgazebo_ros_velodyne_laser.so">
+                <robotNamespace>${robot}</robotNamespace>
                 <topicName>velodyne</topicName>
-                <frameName>lidar</frameName>
+                <frameName>/lidar</frameName>
                 <organize_cloud>false</organize_cloud>
                 <min_range>0.9</min_range>
@@ -222,11 +234,12 @@
     <gazebo> <!-- can't use reference because gazebo squashes fixed joints + links into base_link -->
         <plugin name="imu_plugin" filename="libgazebo_ros_imu.so">
+            <robotNamespace>${robot}</robotNamespace>
             <alwaysOn>true</alwaysOn>
             <bodyName>imu</bodyName>
-            <topicName>/imu</topicName>
+            <topicName>imu</topicName>
             <frameName>imu</frameName>
             <serviceName>imu_service</serviceName>
             <gaussianNoise>0.0</gaussianNoise>
-            <updateRate>20.0</updateRate>
+            <updateRate>50.0</updateRate>
         </plugin>
     </gazebo>
@@ -234,10 +247,11 @@
         <!-- http://wiki.ros.org/hector_gazebo_plugins#GazeboRosGps -->
         <plugin name="gps_controller" filename="libhector_gazebo_ros_gps.so">
+            <robotNamespace>${robot}</robotNamespace>
             <alwaysOn>true</alwaysOn>
             <rosDebugLevel>debug</rosDebugLevel>
             <updateRate>1.0</updateRate>
             <bodyName>base_link</bodyName>
-            <topicName>/fix</topicName> <!-- output topic-->
-            <velocityTopicName>/fix_velocity</velocityTopicName>
+            <topicName>fix</topicName> <!-- output topic-->
+            <velocityTopicName>fix_velocity</velocityTopicName>
             <drift>5.0 5.0 5.0</drift>
             <gaussianNoise>0.1 0.1 0.1</gaussianNoise>
@@ -288,5 +302,5 @@
             <visualize>true</visualize>
             <plugin name="depth_cam_plugin" filename="libgazebo_ros_depth_camera.so">
-                <robotNamespace>choo_choo</robotNamespace>
+                <robotNamespace>${robot}</robotNamespace>
                 <always_on>true</always_on>
                 <updateRate>0.0</updateRate> <!-- use sensor rate -->
@@ -323,5 +337,5 @@
         <plugin name="skid_steer_drive_controller" filename="libgazebo_ros_skid_steer_drive.so">
             <updateRate>100.0</updateRate>
-            <robotNamespace>/</robotNamespace>
+            <robotNamespace>${robot}</robotNamespace>
             <leftFrontJoint>front_left_wheel_joint</leftFrontJoint>
             <rightFrontJoint>front_right_wheel_joint</rightFrontJoint>
@@ -331,9 +345,9 @@
             <wheelDiameter>${wheel_radius * 2}</wheelDiameter>
             <robotBaseFrame>base_link</robotBaseFrame>
-            <torque>20</torque>
-            <commandTopic>cmd_vel</commandTopic>
+            <torque>50</torque>
+            <commandTopic>/cmd_vel</commandTopic>
             <odometryTopic>odom</odometryTopic>
-            <odometryFrame>odom</odometryFrame>
-            <broadcastTF>true</broadcastTF>
+            <odometryFrame>/odom</odometryFrame>
+            <broadcastTF>false</broadcastTF>
         </plugin>
     </gazebo>

Commit message: adjusts model inertias so it can drive

File: ugv_description/urdf/choo_choo/model.urdf.xacro (robot description, xacro)
@@ -4,5 +4,5 @@
     <!-- physical parameters of robot, all in SI (meters, kg) -->
     <!-- base dimensions -->
-    <xacro:property name="base_mass" value="22.67" />
+    <xacro:property name="base_mass" value="45.36" />
     <xacro:property name="base_width" value="0.5588" />     <!-- width=y -->
     <xacro:property name="base_length" value="0.9398" />    <!-- length=x -->
@@ -13,6 +13,6 @@
     <!-- differential properties -->
     <xacro:property name="wheel_mass" value="1.179" />
-    <xacro:property name="wheelbase" value="0.5874" />
-    <xacro:property name="track_width" value="${base_width + (2*0.0994) - 2*(wheel_width/2)}" />
+    <xacro:property name="wheelbase" value="0.67" />
+    <xacro:property name="track_width" value="0.67" />
     <xacro:property name="wheel_offset_x" value="${wheelbase / 2}" />
     <xacro:property name="wheel_offset_y" value="${track_width / 2}" />
@@ -40,5 +40,5 @@
     <xacro:property name="cam_offset_y" value="0.0" />
     <xacro:property name="cam_offset_z" value="${(base_height / 2) + cam_height}" />
-    <xacro:macro name="box" params="name mass width height length">
+    <xacro:macro name="box_total" params="name mass width height length">
         <link name="${name}">
             <gazebo reference="${name}">
@@ -61,7 +61,7 @@
                 <mass value="${mass}" />
                 <!-- 3D inertia tensor from: https://en.wikipedia.org/wiki/List_of_moments_of_inertia -->
-                <inertia ixx="${0.0833*mass*((height*height)+(length*length))}" ixy="0.0" ixz="0.0"
-                        iyy="${0.0833*mass*((height*height)+(width*width))}" iyz="0.0"
-                        izz="${0.0833*mass*((length*length)+(width*width))}" />
+                <inertia ixx="${mass*(height*height+length*length)/12}" ixy="0.0" ixz="0.0"
+                        iyy="${mass*(height*height+width*width)/12}" iyz="0.0"
+                        izz="${mass*(length*length+width*width)/12}" />
             </inertial>
         </link>
@@ -71,7 +71,7 @@
             <mass value="${mass}" />
             <!-- 3D inertia tensor from: https://en.wikipedia.org/wiki/List_of_moments_of_inertia -->
-            <inertia ixx="${0.0833*mass*((height*height)+(length*length))}" ixy="0.0" ixz="0.0"
-                     iyy="${0.0833*mass*((height*height)+(width*width))}" iyz="0.0"
-                     izz="${0.0833*mass*((length*length)+(width*width))}" />
+            <inertia ixx="${mass*((height*height)+(length*length))/12}" ixy="0.0" ixz="0.0"
+                     iyy="${mass*((height*height)+(width*width))/12}" iyz="0.0"
+                     izz="${mass*((length*length)+(width*width))/12}" />
         </inertial>
     </xacro:macro>
@@ -80,7 +80,7 @@
             <mass value="${mass}" />
             <!-- 3D inertia tensor from: https://en.wikipedia.org/wiki/List_of_moments_of_inertia -->
-            <inertia ixx="${0.0833*mass*((height*height)+(3*(radius*radius)))}" ixy="0.0" ixz="0.0"
-                    iyy="${0.0833*mass*((height*height)+(3*(radius*radius)))}" iyz="0.0"
-                    izz="${0.0833*mass*(radius*radius)}" />
+            <inertia ixx="${mass*(height*height+3*radius*radius)/12}" ixy="0.0" ixz="0.0"
+                    iyy="${mass*((height*height)+(3*(radius*radius)))/12}" iyz="0.0"
+                    izz="${mass*(radius*radius)/2}" />
         </inertial>
     </xacro:macro>
@@ -134,5 +134,5 @@
     </gazebo>
     <!-- base link (the box) -->
-    <xacro:box name="base_link" mass="${base_mass}" width="${base_width}" length="${base_length}" height="${base_height}"/>
+    <xacro:box_total name="base_link" mass="${base_mass}" width="${base_width}" length="${base_length}" height="${base_height}"/>
     <!-- front left wheel -->
     <xacro:wheel name="front_left_wheel" wheel_radius="${wheel_radius}" wheel_width="${wheel_width}" wheel_mass="${wheel_mass}"/>
@@ -148,5 +148,5 @@
     <xacro:wheel_joint name="back_right_wheel" x_offset="${wheel_offset_x}" y_offset="${wheel_offset_y}" z_offset="${wheel_offset_z}" reflect_x="-1" reflect_y="-1"/>
     <!-- lidar stalk -->
-    <xacro:box name="lidar_stalk" mass="0.14982" width="${lidar_stalk_side}" length="${lidar_stalk_side}" height="${lidar_stalk_height}" />
+    <xacro:box_total name="lidar_stalk" mass="0.14982" width="${lidar_stalk_side}" length="${lidar_stalk_side}" height="${lidar_stalk_height}" />
     <joint name="lidar_stalk_joint" type="fixed">
         <gazebo reference="lidar_stalk_joint">
@@ -223,5 +223,5 @@
     </gazebo>
     <!-- imu link -->
-    <xacro:box name="imu" mass="0.05" width="0.05" height="0.05" length="0.05"/>
+    <xacro:box_total name="imu" mass="0.05" width="0.05" height="0.05" length="0.05"/>
     <joint name="imu_joint" type="fixed">
         <gazebo reference="imu_joint">
@@ -267,5 +267,5 @@
     </gazebo>
     <!-- stereo camera link -->
-    <xacro:box name="camera" mass="${cam_mass}" width="${cam_width}" length="${cam_length}" height="${cam_height}"/>
+    <xacro:box_total name="camera" mass="${cam_mass}" width="${cam_width}" length="${cam_length}" height="${cam_height}"/>
     <joint name="camera_joint" type="fixed">
         <parent link="base_link"/>
@@ -345,5 +345,5 @@
             <wheelDiameter>${wheel_radius * 2}</wheelDiameter>
             <robotBaseFrame>base_link</robotBaseFrame>
-            <torque>50</torque>
+            <torque>100</torque>
             <commandTopic>/cmd_vel</commandTopic>
             <odometryTopic>odom</odometryTopic>
