Commit message: update to match real vehicle

File: ugv_description/urdf/choo_2/model.urdf.xacro (robot description, xacro)
@@ -82,6 +82,6 @@
     </joint>
     <!-- lidar link -->
-    <link name="lidar">
-        <gazebo reference="lidar">
+    <link name="velodyne">
+        <gazebo reference="velodyne">
         </gazebo>
         <collision>
@@ -97,5 +97,5 @@
             </geometry>
         </visual>
-        <xacro:cylinder_inertia name="lidar" height="${lidar_height}" radius="${lidar_radius}" mass="${lidar_mass}" />
+        <xacro:cylinder_inertia name="velodyne" height="${lidar_height}" radius="${lidar_radius}" mass="${lidar_mass}" />
     </link>
     <joint name="lidar_joint" type="fixed">
@@ -103,14 +103,14 @@
         </gazebo>
         <parent link="lidar_stalk" />
-        <child link="lidar" />
-        <origin xyz="0 0 ${lidar_stalk_height / 2}" />
+        <child link="velodyne" />
+        <origin xyz="0 0 ${lidar_stalk_height / 2}" rpy="0 0 1.5708" />
     </joint>
     <!-- imu link -->
-    <xacro:box_total name="imu" mass="0.05" width="0.05" height="0.05" length="0.05"/>
+    <xacro:box_total name="vectornav" mass="0.05" width="0.05" height="0.05" length="0.05"/>
     <joint name="imu_joint" type="fixed">
         <gazebo reference="imu_joint">
         </gazebo>
         <parent link="base_link"/>
-        <child link="imu"/>
+        <child link="vectornav"/>
         <origin xyz="${imu_offset_x} ${imu_offset_y} ${imu_offset_z}" rpy="0 0 0" />
     </joint>
@@ -121,4 +121,16 @@
         <child link="camera"/>
         <origin xyz="${cam_offset_x} ${cam_offset_y} ${cam_offset_z}" rpy="0 0 0" />
+    </joint>
+    <link name="zed_left_camera_frame"></link>
+    <link name="zed_right_camera_frame"></link>
+    <joint name="zed_left_joint" type="fixed">
+        <parent link="camera"/>
+        <child link="zed_left_camera_frame"/>
+        <origin xyz="0.0  0.0  0.0" rpy="0 0 0"/>
+    </joint>
+    <joint name="zed_right_joint" type="fixed">
+        <parent link="camera"/>
+        <child link="zed_right_camera_frame"/>
+        <origin xyz="0.0  0.0  0.0" rpy="0 0 0"/>
     </joint>
     <!-- a simulation workaround to fix the broken point cloud orientation -->

File: ugv_description/urdf/choo_choo/model.urdf (robot description, URDF)
Before this commit: robot choo_choo, 10 links, 9 joints
Links:
- link back_left_wheel: geometry collision cylinder length=0.059 radius=0.10795; visual cylinder length=0.059 radius=0.10795
- link back_right_wheel: geometry collision cylinder length=0.059 radius=0.10795; visual cylinder length=0.059 radius=0.10795
- link base_link: mass 22.67 -> 45.36
- link front_left_wheel: geometry collision cylinder length=0.059 radius=0.10795; visual cylinder length=0.059 radius=0.10795
- link front_right_wheel: geometry collision cylinder length=0.059 radius=0.10795; visual cylinder length=0.059 radius=0.10795
- link lidar: geometry collision cylinder length=0.0717 radius=0.0516; visual cylinder length=0.0717 radius=0.0516
Joints:
- joint back_left_wheel_joint: origin xyz=-0.2937 0.34829999999999994 -0.186475 -> xyz=-0.335 0.335 -0.186475
- joint back_right_wheel_joint: origin xyz=-0.2937 -0.34829999999999994 -0.186475 -> xyz=-0.335 -0.335 -0.186475
- joint front_left_wheel_joint: origin xyz=0.2937 0.34829999999999994 -0.186475 -> xyz=0.335 0.335 -0.186475
- joint front_right_wheel_joint: origin xyz=0.2937 -0.34829999999999994 -0.186475 -> xyz=0.335 -0.335 -0.186475

File: ugv_description/urdf/choo_choo/model.urdf.xacro (robot description, xacro)
@@ -5,5 +5,5 @@
     <!-- base dimensions -->
     <xacro:property name="base_mass" value="45.36" />
-    <xacro:property name="base_width" value="0.5588" />     <!-- width=y -->
+    <xacro:property name="base_width" value="0.4" />     <!-- width=y -->
     <xacro:property name="base_length" value="0.9398" />    <!-- length=x -->
     <xacro:property name="base_height" value="0.305" />     <!-- height=z -->
@@ -13,6 +13,7 @@
     <!-- differential properties -->
     <xacro:property name="wheel_mass" value="1.179" />
-    <xacro:property name="wheelbase" value="0.67" />
-    <xacro:property name="track_width" value="0.67" />
+    <!-- <xacro:property name="wheelbase" value="0.67" /> -->
+    <xacro:property name="wheelbase" value="0.40" />
+    <xacro:property name="track_width" value="0.54" />
     <xacro:property name="wheel_offset_x" value="${wheelbase / 2}" />
     <xacro:property name="wheel_offset_y" value="${track_width / 2}" />
@@ -345,5 +346,5 @@
             <wheelDiameter>${wheel_radius * 2}</wheelDiameter>
             <robotBaseFrame>base_link</robotBaseFrame>
-            <torque>100</torque>
+            <torque>4</torque>
             <commandTopic>/cmd_vel</commandTopic>
             <odometryTopic>odom</odometryTopic>

Commit message: adds gps_link

File: ugv_description/urdf/choo_2/model.urdf.xacro (robot description, xacro)
@@ -115,4 +115,13 @@
         <origin xyz="${imu_offset_x} ${imu_offset_y} ${imu_offset_z}" rpy="0 0 0" />
     </joint>
+    <!-- gps link -->
+    <xacro:box_total name="gps_link" mass="0.05" width="0.05" height="0.05" length="0.05"/>
+    <joint name="gps_joint" type="fixed">
+        <gazebo reference="gps_joint">
+        </gazebo>
+        <parent link="base_link"/>
+        <child link="gps_link"/>
+        <origin xyz="-0.4249 0 -.09" rpy="0 0 0" />
+    </joint>
     <!-- stereo camera link -->
     <xacro:box_total name="camera" mass="${cam_mass}" width="${cam_width}" length="${cam_length}" height="${cam_height}"/>
